Commit message: Added two versions of URDF exports, both work

File: catkin_ws/src/optimus_corrected_origin/urdf/optimus_corrected_origin.urdf (robot description, URDF)
Before this commit: robot optimus, 19 links, 18 joints
Links:
- link FL_inner_wheel_connector_link: geometry collision mesh filename=package://optimus_corrected_origin/meshes/FL_inner_wheel_co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; visual mesh filename=package://optimus_corrected_origin/meshes/FL_inner_wheel_co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
- link FL_inner_wheel_link: geometry collision mesh filename=package://optimus_corrected_origin/meshes/FL_inner_wheel_li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; visual mesh filename=package://optimus_corrected_origin/meshes/FL_inner_wheel_li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
- link FL_outer_wheel__link: geometry collision mesh filename=package://optimus_corrected_origin/meshes/FL_outer_wheel__l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; visual mesh filename=package://optimus_corrected_origin/meshes/FL_outer_wheel__l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
- link FL_outer_wheel_connector_link: geometry collision mesh filename=package://optimus_corrected_origin/meshes/FL_outer_wheel_co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; visual mesh filename=package://optimus_corrected_origin/meshes/FL_outer_wheel_co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
- link FR_inner_wheel_connector_link: geometry collision mesh filename=package://optimus_corrected_origin/meshes/FR_inner_wheel_co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; visual mesh filename=package://optimus_corrected_origin/meshes/FR_inner_wheel_co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
- link FR_inner_wheel_link: mass 5.00504892402195 -> 5.00504892402194; geometry collision mesh filename=package://optimus_corrected_origin/meshes/FR_inner_wheel_li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; visual mesh filename=package://optimus_corrected_origin/meshes/FR_inner_wheel_li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
- link FR_outer_wheel_connector_link: geometry collision mesh filename=package://optimus_corrected_origin/meshes/FR_outer_wheel_co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; visual mesh filename=package://optimus_corrected_origin/meshes/FR_outer_wheel_co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
- link FR_outer_wheel_link: mass 39.6885330149724 -> 39.6885330149725; geometry collision mesh filename=package://optimus_corrected_origin/meshes/FR_outer_wheel_li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; visual mesh filename=package://optimus_corrected_origin/meshes/FR_outer_wheel_li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
- link F_bogie_link: mass 75.1415926535898 -> 75.142; geometry collision mesh filename=package://optimus_corrected_origin/meshes/F_bogie_link.STL; visual mesh filename=package://optimus_corrected_origin/meshes/F_bogie_link.STL
- link RL_inner_wheel_connector_link: geometry collision mesh filename=package://optimus_corrected_origin/meshes/RL_inner_wheel_co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; visual mesh filename=package://optimus_corrected_origin/meshes/RL_inner_wheel_co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
- link RL_inner_wheel_link: geometry collision mesh filename=package://optimus_corrected_origin/meshes/RL_inner_wheel_li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; visual mesh filename=package://optimus_corrected_origin/meshes/RL_inner_wheel_li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
- link RL_outer_wheel_connector_link: geometry collision mesh filename=package://optimus_corrected_origin/meshes/RL_outer_wheel_co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; visual mesh filename=package://optimus_corrected_origin/meshes/RL_outer_wheel_co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
- link RL_outer_wheel_link: geometry collision mesh filename=package://optimus_corrected_origin/meshes/RL_outer_wheel_li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; visual mesh filename=package://optimus_corrected_origin/meshes/RL_outer_wheel_li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
- link RR_inner_wheel_connector_link: geometry collision mesh filename=package://optimus_corrected_origin/meshes/RR_inner_wheel_co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; visual mesh filename=package://optimus_corrected_origin/meshes/RR_inner_wheel_co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
- link RR_inner_wheel_link: geometry collision mesh filename=package://optimus_corrected_origin/meshes/RR_inner_wheel_li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; visual mesh filename=package://optimus_corrected_origin/meshes/RR_inner_wheel_li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
- link RR_outer_wheel_connector_link: geometry collision mesh filename=package://optimus_corrected_origin/meshes/RR_outer_wheel_co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; visual mesh filename=package://optimus_corrected_origin/meshes/RR_outer_wheel_co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
- link RR_outer_wheel_link: geometry collision mesh filename=package://optimus_corrected_origin/meshes/RR_outer_wheel_li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; visual mesh filename=package://optimus_corrected_origin/meshes/RR_outer_wheel_li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
- link R_bogie_link: geometry collision mesh filename=package://optimus_corrected_origin/meshes/R_bogie_link.STL; visual mesh filename=package://optimus_corrected_origin/meshes/R_bogie_link.STL
- link base_link: mass 144.386284511659 -> 144.39; geometry collision mesh filename=package://optimus_corrected_origin/meshes/base_link.STL; visual mesh filename=package://optimus_corrected_origin/meshes/base_link.STL
Joints:
- joint FL_inner_wheel_connector_joint: origin xyz=0.15 0.265 -0.09 rpy=1.5708 0 1.5708 -> xyz=0.15 0.265 -0.1 rpy=0 0 0
- joint FL_inner_wheel_joint: axis 1 0 0 -> 0 -1 0; origin xyz=-0.0250000000000001 -1.82399954632428E-05 0.319396288800974 rpy=-3.08118480125405 0 3.14159265358979 -> xyz=0.32 -0.025 0 rpy=0 0 0
- joint FL_outer_wheel_connector_joint: axis 0 0 1 -> 0 0 0; origin xyz=0.191410490599822 -0.0151205788993285 0 rpy=3.14159265358979 0 -1.03321742493139 -> xyz=0.2 -0.3 -0.1 rpy=0 0 0; type continuous -> fixed
- joint FL_outer_wheel_joint: axis 1 0 0 -> 0 -1 0; origin xyz=0.0096055118553634 -0.00721896745857198 0.326743890579708 rpy=1.85261522674577 -1.5707963267949 0 -> xyz=0 -0.32674 0 rpy=0 0 0
- joint FR_inner_wheel_connector_joint: origin xyz=0.15 -0.265 -0.11 rpy=-1.5708 0 -1.5708 -> xyz=0.15 -0.265 -0.1 rpy=0 0 0
- joint FR_inner_wheel_joint: axis 1 0 0 -> 0 1 0; origin xyz=-0.0249999999999999 -0.00410574285570231 0.328078225839681 rpy=2.2011440774755 0 3.14159265358979 -> xyz=0.32 0.025 0 rpy=0 0 0
- joint FR_outer_wheel_connector_joint: axis 0 0 1 -> 0 0 0; origin xyz=0.20965 -0.0073618 0.6 rpy=0 0 -1.3038 -> xyz=0.2 0.3 -0.1 rpy=0 0 0; type continuous -> fixed
- joint FR_outer_wheel_joint: axis 1 0 0 -> 0 1 0; origin xyz=0.0096055 -0.007219 0.32674 rpy=1.8526 -1.5708 0 -> xyz=0 0.32674 0 rpy=0 0 0
- joint F_bogie_joint: origin xyz=1.1 -0.3 -0.11 rpy=-1.5708 0 0 -> xyz=1.1 0 0 rpy=0 0 0
- joint RL_inner_wheel_connector_joint: origin xyz=-0.15 0.265 -0.11 rpy=-1.5708 0 1.5708 -> xyz=-0.15 0.265 -0.1 rpy=0 0 0
- joint RL_inner_wheel_joint: axis 0 0 1 -> 0 -1 0; origin xyz=-0.0249999999999979 -0.00913637272663603 0.329962637599185 rpy=1.5707963267949 -0.0864704456326401 -1.5707963267949 -> xyz=-0.32 -0.025 0 rpy=0 0 0
- joint RL_outer_wheel_connector_joint: axis 0 0 1 -> 0 0 0; origin xyz=0.19018 -0.0081271 -0.6 rpy=3.1416 0 -1.7592 -> xyz=-0.2 0.3 -0.1 rpy=0 0 0; type continuous -> fixed
- joint RL_outer_wheel_joint: axis 1 0 0 -> 0 1 0; origin xyz=0.00960551185536335 -0.00721896745857231 0.326743890579709 rpy=1.85261522674576 -1.5707963267949 0 -> xyz=0 0.32674 0 rpy=0 0 0
- joint RR_inner_wheel_connector_joint: origin xyz=-0.149999999999999 -0.265 -0.0899999999999999 rpy=1.5707963267949 0 -1.5707963267949 -> xyz=-0.15 -0.265 -0.1 rpy=0 0 0
- joint RR_inner_wheel_joint: axis 0 0 1 -> 0 1 0; origin xyz=-0.0249999999999991 -0.00250756059284885 0.326622941320151 rpy=1.5707963267949 -0.846919764335258 -1.5707963267949 -> xyz=-0.32 0.025 0 rpy=0 0 0
- joint RR_outer_wheel_connector_joint: axis 0 0 1 -> 0 0 0; origin xyz=0.20777741525486 -0.0162858421833096 0 rpy=0 0 -2.25052782068816 -> xyz=-0.2 -0.3 -0.1 rpy=0 0 0; type continuous -> fixed
- joint RR_outer_wheel_joint: axis 1 0 0 -> 0 -1 0; origin xyz=0.0096055118553634 -0.00721896745857276 0.326743890579708 rpy=1.85261522674574 -1.5707963267949 0 -> xyz=0 -0.32674 0 rpy=0 0 0
- joint R_bogie_joint: origin xyz=-1.1 -0.3 -0.109999999999998 rpy=-1.5707963267949 0 -3.14159265358979 -> xyz=-1.1 0 0 rpy=0 0 0

File: catkin_ws/src/optimus_no_origin_change/urdf/optimus_no_origin_change.urdf (robot description, URDF)
Before this commit: robot optimus, 19 links, 18 joints
Links:
- link FL_inner_wheel_connector_link: geometry collision mesh filename=package://optimus_no_origin_change/meshes/FL_inner_wheel_co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; visual mesh filename=package://optimus_no_origin_change/meshes/FL_inner_wheel_co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
- link FL_inner_wheel_link: geometry collision mesh filename=package://optimus_no_origin_change/meshes/FL_inner_wheel_li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; visual mesh filename=package://optimus_no_origin_change/meshes/FL_inner_wheel_li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
- link FL_outer_wheel__link: geometry collision mesh filename=package://optimus_no_origin_change/meshes/FL_outer_wheel__l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; visual mesh filename=package://optimus_no_origin_change/meshes/FL_outer_wheel__l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
- link FL_outer_wheel_connector_link: geometry collision mesh filename=package://optimus_no_origin_change/meshes/FL_outer_wheel_co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; visual mesh filename=package://optimus_no_origin_change/meshes/FL_outer_wheel_co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
- link FR_inner_wheel_connector_link: geometry collision mesh filename=package://optimus_no_origin_change/meshes/FR_inner_wheel_co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; visual mesh filename=package://optimus_no_origin_change/meshes/FR_inner_wheel_co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
- link FR_inner_wheel_link: mass 5.00504892402195 -> 5.00504892402194; geometry collision mesh filename=package://optimus_no_origin_change/meshes/FR_inner_wheel_li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; visual mesh filename=package://optimus_no_origin_change/meshes/FR_inner_wheel_li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
- link FR_outer_wheel_connector_link: geometry collision mesh filename=package://optimus_no_origin_change/meshes/FR_outer_wheel_co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; visual mesh filename=package://optimus_no_origin_change/meshes/FR_outer_wheel_co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
- link FR_outer_wheel_link: mass 39.6885330149724 -> 39.6885330149725; geometry collision mesh filename=package://optimus_no_origin_change/meshes/FR_outer_wheel_li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; visual mesh filename=package://optimus_no_origin_change/meshes/FR_outer_wheel_li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
- link F_bogie_link: geometry collision mesh filename=package://optimus_no_origin_change/meshes/F_bogie_link.STL; visual mesh filename=package://optimus_no_origin_change/meshes/F_bogie_link.STL
- link RL_inner_wheel_connector_link: geometry collision mesh filename=package://optimus_no_origin_change/meshes/RL_inner_wheel_co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; visual mesh filename=package://optimus_no_origin_change/meshes/RL_inner_wheel_co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
- link RL_inner_wheel_link: geometry collision mesh filename=package://optimus_no_origin_change/meshes/RL_inner_wheel_li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; visual mesh filename=package://optimus_no_origin_change/meshes/RL_inner_wheel_li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
- link RL_outer_wheel_connector_link: geometry collision mesh filename=package://optimus_no_origin_change/meshes/RL_outer_wheel_co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; visual mesh filename=package://optimus_no_origin_change/meshes/RL_outer_wheel_co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
- link RL_outer_wheel_link: geometry collision mesh filename=package://optimus_no_origin_change/meshes/RL_outer_wheel_li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; visual mesh filename=package://optimus_no_origin_change/meshes/RL_outer_wheel_li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
- link RR_inner_wheel_connector_link: geometry collision mesh filename=package://optimus_no_origin_change/meshes/RR_inner_wheel_co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; visual mesh filename=package://optimus_no_origin_change/meshes/RR_inner_wheel_co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
- link RR_inner_wheel_link: geometry collision mesh filename=package://optimus_no_origin_change/meshes/RR_inner_wheel_li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; visual mesh filename=package://optimus_no_origin_change/meshes/RR_inner_wheel_li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
- link RR_outer_wheel_connector_link: geometry collision mesh filename=package://optimus_no_origin_change/meshes/RR_outer_wheel_co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; visual mesh filename=package://optimus_no_origin_change/meshes/RR_outer_wheel_co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
- link RR_outer_wheel_link: geometry collision mesh filename=package://optimus_no_origin_change/meshes/RR_outer_wheel_li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; visual mesh filename=package://optimus_no_origin_change/meshes/RR_outer_wheel_li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
- link R_bogie_link: geometry collision mesh filename=package://optimus_no_origin_change/meshes/R_bogie_link.STL; visual mesh filename=package://optimus_no_origin_change/meshes/R_bogie_link.STL
- link base_link: geometry collision mesh filename=package://optimus_no_origin_change/meshes/base_link.STL; visual mesh filename=package://optimus_no_origin_change/meshes/base_link.STL
Joints:
- joint FL_inner_wheel_connector_joint: origin xyz=0.15 0.265 -0.09 rpy=1.5708 0 1.5708 -> xyz=0.15 0.265 -0.1 rpy=1.5708 0 1.5708
- joint FL_inner_wheel_joint: origin xyz=-0.0250000000000001 -1.82399954632428E-05 0.319396288800974 rpy=-3.08118480125405 0 3.14159265358979 -> xyz=-0.0250000000000001 0 0.32 rpy=-3.08118480125405 0 3.14159265358979
- joint FL_outer_wheel_connector_joint: axis 0 0 1 -> 0 0 0; origin xyz=0.191410490599822 -0.0151205788993285 0 rpy=3.14159265358979 0 -1.03321742493139 -> xyz=0.2 0 0 rpy=3.1416 0 -1.0332; type continuous -> fixed
- joint FL_outer_wheel_joint: origin xyz=0.0096055118553634 -0.00721896745857198 0.326743890579708 rpy=1.85261522674577 -1.5707963267949 0 -> xyz=0 0 0.326743890579708 rpy=1.85261522674577 -1.5707963267949 0
- joint FR_inner_wheel_connector_joint: origin xyz=0.15 -0.265 -0.11 rpy=-1.5708 0 -1.5708 -> xyz=0.15 -0.265 -0.1 rpy=-1.5708 0 -1.5708
- joint FR_inner_wheel_joint: origin xyz=-0.0249999999999999 -0.00410574285570231 0.328078225839681 rpy=2.2011440774755 0 3.14159265358979 -> xyz=-0.0249999999999999 0 0.32 rpy=2.2011440774755 0 3.14159265358979
- joint FR_outer_wheel_connector_joint: axis 0 0 1 -> 0 0 0; origin xyz=0.20965 -0.0073618 0.6 rpy=0 0 -1.3038 -> xyz=0.2 0 0.6 rpy=0 0 -1.3038; type continuous -> fixed
- joint FR_outer_wheel_joint: origin xyz=0.0096055 -0.007219 0.32674 rpy=1.8526 -1.5708 0 -> xyz=0 0 0.326743890579709 rpy=1.85261522674577 -1.5707963267949 0
- joint F_bogie_joint: origin xyz=1.1 -0.3 -0.11 rpy=-1.5708 0 0 -> xyz=1.1 -0.3 -0.1 rpy=-1.5707963267949 0 0
- joint RL_inner_wheel_connector_joint: origin xyz=-0.15 0.265 -0.11 rpy=-1.5708 0 1.5708 -> xyz=-0.15 0.265 -0.1 rpy=-1.5708 0 1.5708
- joint RL_inner_wheel_joint: origin xyz=-0.0249999999999979 -0.00913637272663603 0.329962637599185 rpy=1.5707963267949 -0.0864704456326401 -1.5707963267949 -> xyz=-0.0249999999999979 0 0.32 rpy=1.5707963267949 -0.0864704456326401 -1.5707963267949
- joint RL_outer_wheel_connector_joint: axis 0 0 1 -> 0 0 0; origin xyz=0.19018 -0.0081271 -0.6 rpy=3.1416 0 -1.7592 -> xyz=0.2 0 -0.6 rpy=3.1416 0 -1.7592; type continuous -> fixed
- joint RL_outer_wheel_joint: origin xyz=0.00960551185536335 -0.00721896745857231 0.326743890579709 rpy=1.85261522674576 -1.5707963267949 0 -> xyz=0 0 0.326743890579709 rpy=1.85261522674576 -1.5707963267949 0
- joint RR_inner_wheel_connector_joint: origin xyz=-0.149999999999999 -0.265 -0.0899999999999999 rpy=1.5707963267949 0 -1.5707963267949 -> xyz=-0.149999999999999 -0.265 -0.0999999999999999 rpy=1.5707963267949 0 -1.5707963267949
- joint RR_inner_wheel_joint: origin xyz=-0.0249999999999991 -0.00250756059284885 0.326622941320151 rpy=1.5707963267949 -0.846919764335258 -1.5707963267949 -> xyz=-0.0249999999999991 0 0.32 rpy=1.5707963267949 -0.846919764335258 -1.5707963267949
- joint RR_outer_wheel_connector_joint: axis 0 0 1 -> 0 0 0; origin xyz=0.20777741525486 -0.0162858421833096 0 rpy=0 0 -2.25052782068816 -> xyz=0.2 0 0 rpy=0 0 -2.2505; type continuous -> fixed
- joint RR_outer_wheel_joint: origin xyz=0.0096055118553634 -0.00721896745857276 0.326743890579708 rpy=1.85261522674574 -1.5707963267949 0 -> xyz=0 0 0.326743890579708 rpy=1.85261522674574 -1.5707963267949 0
- joint R_bogie_joint: origin xyz=-1.1 -0.3 -0.109999999999998 rpy=-1.5707963267949 0 -3.14159265358979 -> xyz=-1.1 -0.3 -0.0999999999999984 rpy=-1.5707963267949 0 -3.14159265358979
