Commit message: Backup before changing URDFs

File: catkin_ws/src/optimus_front/urdf/optimus_front.urdf.xacro (robot description, xacro)
@@ -4,5 +4,6 @@
      For more information, please see http://wiki.ros.org/sw_urdf_exporter -->
 <robot
-  name="optimus_front">
+  name="optimus_front" xmlns:xacro="http://ros.org/wiki/xacro">
+  <xacro:include filename="$(find optimus_front)/urdf/optimus_front.gazebo" />
   <link
     name="optimus_front">
@@ -98,9 +99,19 @@
       xyz="0 1 0" />
     <limit
-      lower="0"
+      lower="1.57"
       upper="0"
-      effort="0"
-      velocity="0" />
-  </joint>
+      effort="10"
+      velocity="10" />
+  </joint>
+  <transmission name="FR_outer_wheel_connector_trans">
+    <type>transmission_interface/SimpleTransmission</type>
+    <joint name="FR_outer_wheel_connector_joint">
+      <hardwareInterface>hardware_interface/PositionJointInterface</hardwareInterface>
+    </joint>
+    <actuator name="FR_outer_wheel_connector_actuator">
+      <mechanicalReduction>1</mechanicalReduction>
+      <hardwareInterface>hardware_interface/PositionJointInterface</hardwareInterface>
+    </actuator>
+  </transmission>
   <link
     name="FR_outer_wheel_link">
@@ -154,6 +165,16 @@
       link="FR_outer_wheel_link" />
     <axis
-      xyz="0 -1 0" />
-  </joint>
+      xyz="0 1 0" />
+  </joint>
+  <transmission name="FR_outer_wheel_trans">
+    <type>transmission_interface/SimpleTransmission</type>
+    <joint name="FR_outer_wheel_joint">
+      <hardwareInterface>hardware_interface/VelocityJointInterface</hardwareInterface>
+    </joint>
+    <actuator name="FR_outer_wheel_actuator">
+      <mechanicalReduction>1</mechanicalReduction>
+      <hardwareInterface>hardware_interface/VelocityJointInterface</hardwareInterface>
+    </actuator>
+  </transmission>
   <link
     name="FL_outer_wheel_connector_link">
@@ -211,7 +232,17 @@
       lower="0"
       upper="0"
-      effort="0"
-      velocity="0" />
-  </joint>
+      effort="10"
+      velocity="10" />
+  </joint>
+  <transmission name="FL_outer_wheel_connector_trans">
+    <type>transmission_interface/SimpleTransmission</type>
+    <joint name="FL_outer_wheel_connector_joint">
+      <hardwareInterface>hardware_interface/PositionJointInterface</hardwareInterface>
+    </joint>
+    <actuator name="FL_outer_wheel_connector_actuator">
+      <mechanicalReduction>1</mechanicalReduction>
+      <hardwareInterface>hardware_interface/PositionJointInterface</hardwareInterface>
+    </actuator>
+  </transmission>
   <link
     name="FL_outer_wheel_link">
@@ -267,4 +298,14 @@
       xyz="0 1 0" />
   </joint>
+  <transmission name="FL_outer_wheel_trans">
+    <type>transmission_interface/SimpleTransmission</type>
+    <joint name="FL_outer_wheel_joint">
+      <hardwareInterface>hardware_interface/VelocityJointInterface</hardwareInterface>
+    </joint>
+    <actuator name="FL_outer_wheel_actuator">
+      <mechanicalReduction>1</mechanicalReduction>
+      <hardwareInterface>hardware_interface/VelocityJointInterface</hardwareInterface>
+    </actuator>
+  </transmission>
   <link
     name="FR_inner_wheel_connector_link">
@@ -322,7 +363,17 @@
       lower="0"
       upper="0"
-      effort="0"
-      velocity="0" />
-  </joint>
+      effort="10"
+      velocity="10" />
+  </joint>
+  <transmission name="FR_inner_wheel_connector_trans">
+    <type>transmission_interface/SimpleTransmission</type>
+    <joint name="FR_inner_wheel_connector_joint">
+      <hardwareInterface>hardware_interface/PositionJointInterface</hardwareInterface>
+    </joint>
+    <actuator name="FR_inner_wheel_connector_actuator">
+      <mechanicalReduction>1</mechanicalReduction>
+      <hardwareInterface>hardware_interface/PositionJointInterface</hardwareInterface>
+    </actuator>
+  </transmission>
   <link
     name="FR_inner_wheel_link">
@@ -376,6 +427,16 @@
       link="FR_inner_wheel_link" />
     <axis
-      xyz="0 -1 0" />
-  </joint>
+      xyz="0 1 0" />
+  </joint>
+  <transmission name="FR_inner_wheel_trans">
+    <type>transmission_interface/SimpleTransmission</type>
+    <joint name="FR_inner_wheel_joint">
+      <hardwareInterface>hardware_interface/VelocityJointInterface</hardwareInterface>
+    </joint>
+    <actuator name="FR_inner_wheel_actuator">
+      <mechanicalReduction>1</mechanicalReduction>
+      <hardwareInterface>hardware_interface/VelocityJointInterface</hardwareInterface>
+    </actuator>
+  </transmission>
   <link
     name="FL_inner_wheel_connector_link">
@@ -429,11 +490,21 @@
       link="FL_inner_wheel_connector_link" />
     <axis
-      xyz="0 -1 0" />
+      xyz="0 1 0" />
     <limit
       lower="0"
       upper="0"
-      effort="0"
-      velocity="0" />
-  </joint>
+      effort="10"
+      velocity="10" />
+  </joint>
+  <transmission name="FL_inner_wheel_connector_trans">
+    <type>transmission_interface/SimpleTransmission</type>
+    <joint name="FL_inner_wheel_connector_joint">
+      <hardwareInterface>hardware_interface/PositionJointInterface</hardwareInterface>
+    </joint>
+    <actuator name="FL_inner_wheel_connector_actuator">
+      <mechanicalReduction>1</mechanicalReduction>
+      <hardwareInterface>hardware_interface/PositionJointInterface</hardwareInterface>
+    </actuator>
+  </transmission>
   <link
     name="FL_inner_wheel_link">
@@ -489,4 +560,14 @@
       xyz="0 1 0" />
   </joint>
+  <transmission name="FL_inner_wheel_trans">
+    <type>transmission_interface/SimpleTransmission</type>
+    <joint name="FL_inner_wheel_joint">
+      <hardwareInterface>hardware_interface/VelocityJointInterface</hardwareInterface>
+    </joint>
+    <actuator name="FL_inner_wheel_actuator">
+      <mechanicalReduction>1</mechanicalReduction>
+      <hardwareInterface>hardware_interface/VelocityJointInterface</hardwareInterface>
+    </actuator>
+  </transmission>
   <link
     name="docker_link">
@@ -595,8 +676,8 @@
       xyz="0 0 1" />
     <limit
-      lower="-1"
+      lower="-0.2"
       upper="0"
-      effort="0"
-      velocity="0" />
+      effort="10"
+      velocity="10" />
   </joint>
   <link
@@ -653,8 +734,8 @@
       xyz="0 0 1" />
     <limit
-      lower="-1"
+      lower="-0.2"
       upper="0"
-      effort="0"
-      velocity="0" />
+      effort="10"
+      velocity="10" />
   </joint>
 </robot>

File: catkin_ws/src/optimus_rear/urdf/optimus_rear.urdf.xacro (robot description, xacro)
@@ -4,5 +4,5 @@
      For more information, please see http://wiki.ros.org/sw_urdf_exporter -->
 <robot
-  name="optimus_rear">
+  name="optimus_rear" xmlns:xacro="http://ros.org/wiki/xacro">
   <link
     name="optimus_rear">
@@ -98,5 +98,5 @@
       xyz="0 -1 0" />
     <limit
-      lower="0"
+      lower="1.57"
       upper="0"
       effort="0"
@@ -154,5 +154,5 @@
       link="RR_outer_wheel_link" />
     <axis
-      xyz="0 -1 0" />
+      xyz="0 1 0" />
   </joint>
   <link
@@ -209,5 +209,5 @@
       xyz="0 -1 0" />
     <limit
-      lower="0"
+      lower="1.57"
       upper="0"
       effort="0"
@@ -318,7 +318,7 @@
       link="RR_inner_wheel_connector_link" />
     <axis
-      xyz="0 1 0" />
+      xyz="0 -1 0" />
     <limit
-      lower="0"
+      lower="1.57"
       upper="0"
       effort="0"
@@ -376,5 +376,5 @@
       link="RR_inner_wheel_link" />
     <axis
-      xyz="0 -1 0" />
+      xyz="0 1 0" />
   </joint>
   <link
@@ -431,5 +431,5 @@
       xyz="0 -1 0" />
     <limit
-      lower="0"
+      lower="1.57"
       upper="0"
       effort="0"
