Commit message: Backup before switching to different URDFs, all whels down

File: catkin_ws/src/optimus/urdf/optimus.urdf.xacro (robot description, xacro)
@@ -12,12 +12,13 @@
   </link>
   <joint name="base_optimus_front_joint" type="fixed">
-    <origin xyz="0.5 0 0" rpy="0 0 0" />
+    <origin xyz="0.5 0 -0.44" rpy="0 0 0" />
     <parent link="base_link"/>
     <child link="optimus_front" />
   </joint>
   <joint name="base_optimus_rear_joint" type="fixed">
-    <origin xyz="-0.5 0 0" rpy="0 0 0" />
+    <origin xyz="-0.5 0 -0.44" rpy="0 0 0" />
     <parent link="base_link"/>
     <child link="optimus_rear" />
   </joint>
+  <xacro:include filename="$(find optimus)/urdf/optimus.gazebo" />
 </robot>

File: catkin_ws/src/optimus_front/urdf/optimus_front.urdf.xacro (robot description, xacro)
@@ -5,5 +5,4 @@
 <robot
   name="optimus_front" xmlns:xacro="http://ros.org/wiki/xacro">
-  <xacro:include filename="$(find optimus_front)/urdf/optimus_front.gazebo" />
   <link
     name="optimus_front">
@@ -739,3 +738,4 @@
       velocity="10" />
   </joint>
+  <!-- <xacro:include filename="$(find optimus_front)/urdf/optimus_front.gazebo" /> -->
 </robot>

File: catkin_ws/src/optimus_rear/urdf/optimus_rear.urdf.xacro (robot description, xacro)
@@ -98,5 +98,5 @@
       xyz="0 -1 0" />
     <limit
-      lower="1.57"
+      lower="0"
       upper="0"
       effort="0"
@@ -209,5 +209,5 @@
       xyz="0 -1 0" />
     <limit
-      lower="1.57"
+      lower="0"
       upper="0"
       effort="0"
@@ -320,5 +320,5 @@
       xyz="0 -1 0" />
     <limit
-      lower="1.57"
+      lower="0"
       upper="0"
       effort="0"
@@ -431,5 +431,5 @@
       xyz="0 -1 0" />
     <limit
-      lower="1.57"
+      lower="0"
       upper="0"
       effort="0"
@@ -489,3 +489,4 @@
       xyz="0 1 0" />
   </joint>
+  <!-- <xacro:include filename="$(find optimus_rear)/urdf/optimus_rear.gazebo" /> -->
 </robot>

Commit message: Added controllers to optimus_front_down, Gazebo and RViz work

File: catkin_ws/src/optimus/urdf/optimus.urdf.xacro (robot description, xacro)
@@ -3,7 +3,7 @@
   name="optimus" xmlns:xacro="http://ros.org/wiki/xacro">
   <!-- Importing Optimus Front -->
-  <xacro:include filename="$(find optimus_front)/urdf/optimus_front.urdf.xacro" />
+  <xacro:include filename="$(find optimus_front_down)/urdf/optimus_front_down.urdf" />
   <!-- Importing Optimus Rear -->
-  <xacro:include filename="$(find optimus_rear)/urdf/optimus_rear.urdf.xacro" />
+  <xacro:include filename="$(find optimus_rear_down)/urdf/optimus_rear_down.urdf" />
   <!-- Bring in simulation data for Gazebo. -->
   <!-- <xacro:include filename="$(find optimus_corrected_origin)/urdf/optimus_corrected_origin.gazebo" /> -->
@@ -12,12 +12,12 @@
   </link>
   <joint name="base_optimus_front_joint" type="fixed">
-    <origin xyz="0.5 0 -0.44" rpy="0 0 0" />
+    <origin xyz="0.5 0 0" rpy="0 0 0" />
     <parent link="base_link"/>
-    <child link="optimus_front" />
+    <child link="optimus_front_down" />
   </joint>
   <joint name="base_optimus_rear_joint" type="fixed">
-    <origin xyz="-0.5 0 -0.44" rpy="0 0 0" />
+    <origin xyz="-0.5 0 0" rpy="0 0 0" />
     <parent link="base_link"/>
-    <child link="optimus_rear" />
+    <child link="optimus_rear_down" />
   </joint>
   <xacro:include filename="$(find optimus)/urdf/optimus.gazebo" />

File: catkin_ws/src/optimus_front_down/urdf/optimus_front_down.urdf (robot description, URDF)
Before this commit: robot optimus_front_down, 12 links, 11 joints
Links:
- removed link base_link
- added link optimus_front_down, mass 122.44; collision mesh filename=package://optimus_front_down/meshes/optimus_front_down.STL; visual mesh filename=package://optimus_front_down/meshes/optimus_front_down.STL
Joints:
- joint FL_inner_wheel_connector_joint: limit lower=0 upper=0 effort=0 velocity=0 -> lower=0 upper=1.57 effort=100 velocity=100; parent base_link -> optimus_front_down
- joint FL_outer_wheel_connector_joint: limit lower=0 upper=0 effort=0 velocity=0 -> lower=0 upper=1.57 effort=100 velocity=100; parent base_link -> optimus_front_down
- joint FR_inner_wheel_connector_joint: axis 0 1 0 -> 0 -1 0; limit lower=0 upper=0 effort=0 velocity=0 -> lower=0 upper=1.57 effort=100 velocity=100; parent base_link -> optimus_front_down
- joint FR_inner_wheel_joint: axis 0 -1 0 -> 0 1 0
- joint FR_outer_wheel_connector_joint: limit lower=0.0 upper=1.57 effort=10.0 velocity=10.0 -> lower=0.0 upper=1.57 effort=100 velocity=100; parent base_link -> optimus_front_down
- joint FR_outer_wheel_joint: axis 0 -1 0 -> 0 1 0
- joint L_docker_shaft_joint: limit lower=0 upper=0 effort=0 velocity=0 -> lower=-0.2 upper=0 effort=0 velocity=0
- joint R_docker_shaft_joint: limit lower=0 upper=0 effort=0 velocity=0 -> lower=-0.2 upper=0 effort=10 velocity=10
- joint docker_joint: parent base_link -> optimus_front_down

File: catkin_ws/src/optimus_rear_down/urdf/optimus_rear_down.urdf (robot description, URDF)
Before this commit: robot optimus_rear_down, 9 links, 8 joints
Links:
- removed link base_link
- added link optimus_rear_down, mass 122.376866884981; collision mesh filename=package://optimus_rear_down/meshes/optimus_rear_down.STL; visual mesh filename=package://optimus_rear_down/meshes/optimus_rear_down.STL
Joints:
- joint RL_inner_wheel_connector_joint: axis 0 -1 0 -> 0 1 0; limit lower=0 upper=0 effort=0 velocity=0 -> lower=0 upper=1.57 effort=100 velocity=100; parent base_link -> optimus_rear_down
- joint RL_outer_wheel_connector_joint: limit lower=0 upper=0 effort=0 velocity=0 -> lower=0 upper=1.57 effort=100 velocity=100; parent base_link -> optimus_rear_down
- joint RR_inner_wheel_connector_joint: limit lower=0 upper=0 effort=0 velocity=0 -> lower=0 upper=1.57 effort=100 velocity=100; parent base_link -> optimus_rear_down
- joint RR_inner_wheel_joint: axis 0 -1 0 -> 0 1 0
- joint RR_outer_wheel_connector_joint: limit lower=0 upper=1.57 effort=10 velocity=10 -> lower=0 upper=1.57 effort=100 velocity=100; parent base_link -> optimus_rear_down
- joint RR_outer_wheel_joint: axis 0 -1 0 -> 0 1 0

Commit message: Works but doesn't attach

File: catkin_ws/src/optimus/urdf/optimus.urdf.xacro (robot description, xacro)
@@ -6,6 +6,4 @@
   <!-- Importing Optimus Rear -->
   <xacro:include filename="$(find optimus_rear_down)/urdf/optimus_rear_down.urdf" />
-  <!-- Bring in simulation data for Gazebo. -->
-  <!-- <xacro:include filename="$(find optimus_corrected_origin)/urdf/optimus_corrected_origin.gazebo" /> -->
   <link
     name="base_link">
@@ -21,4 +19,5 @@
     <child link="optimus_rear_down" />
   </joint>
+  <!-- Bring in simulation data for Gazebo. -->
   <xacro:include filename="$(find optimus)/urdf/optimus.gazebo" />
 </robot>

File: catkin_ws/src/optimus_front_down/urdf/optimus_front_down.urdf (robot description, URDF)
Before this commit: robot optimus_front_down, 12 links, 11 joints
Joints:
- joint L_docker_shaft_joint: limit lower=-0.2 upper=0 effort=0 velocity=0 -> lower=-0.2 upper=0.1 effort=10 velocity=10
- joint R_docker_shaft_joint: limit lower=-0.2 upper=0 effort=10 velocity=10 -> lower=-0.2 upper=0.1 effort=10 velocity=10

Commit message: UR10e control works, added gripper

File: catkin_ws/src/optimus/urdf/optimus.urdf.xacro (robot description, xacro)
@@ -3,7 +3,7 @@
   name="optimus" xmlns:xacro="http://ros.org/wiki/xacro">
   <!-- Importing Optimus Front -->
-  <xacro:include filename="$(find optimus_front_down)/urdf/optimus_front_down.urdf" />
+  <xacro:include filename="$(find optimus_front_down)/urdf/optimus_front_down.urdf.xacro" />
   <!-- Importing Optimus Rear -->
-  <xacro:include filename="$(find optimus_rear_down)/urdf/optimus_rear_down.urdf" />
+  <xacro:include filename="$(find optimus_rear_down)/urdf/optimus_rear_down.urdf.xacro" />
   <link
     name="base_link">

File: catkin_ws/src/optimus_front_down/urdf/optimus_front_down.urdf.xacro (robot description, xacro)
@@ -4,5 +4,5 @@
      For more information, please see http://wiki.ros.org/sw_urdf_exporter -->
 <robot
-  name="optimus_front_down">
+  name="optimus_front_down" xmlns:xacro="http://ros.org/wiki/xacro">
   <link
     name="optimus_front_down">
@@ -770,4 +770,17 @@
     </actuator>
   </transmission>
+  <!-- Importing UR_10 -->
+  <!-- <xacro:include filename="$(find ur_e_description)/urdf/common.gazebo.xacro" /> -->
+  <xacro:include filename="$(find ur_e_description)/urdf/ur10e.urdf.xacro" />
+  <xacro:ur10e_robot prefix="ur10e_front_" joint_limited="false"/>
+  <!-- <xacro:include filename="$(find ur_e_description)/urdf/arm_extras_ur10.urdf.xacro" />
+  <xacro:include filename="$(find ur_e_description)/urdf/rg2.urdf.xacro" />
+  <xacro:arm_extras prefix="ur10e_front_" joint_limited="false" kinect_prefix="ur10e_front_kinetic"/>
+  <xacro:rg2 prefix="ur10e_front_"/> -->
+  <joint name="ur10_front_joint" type="fixed">
+    <origin xyz="0.3 0 0.1" rpy="0 0 0" />
+    <parent link="optimus_front_down"/>
+    <child link="ur10e_front_base_link" />
+  </joint>
   <gazebo>
     <plugin filename="libgazebo_ros_control.so" name="gazebo_ros_control">
@@ -778,3 +791,39 @@
     </plugin>
   </gazebo>
+  <gazebo reference="optimus_front_down">
+    <material>Gazebo/Grey</material>
+  </gazebo>
+  <gazebo reference="FR_outer_wheel_link">
+    <material>Gazebo/DarkGrey</material>
+  </gazebo>
+  <gazebo reference="FL_outer_wheel_link">
+    <material>Gazebo/DarkGrey</material>
+  </gazebo>
+  <gazebo reference="FR_inner_wheel_link">
+    <material>Gazebo/DarkGrey</material>
+  </gazebo>
+  <gazebo reference="FL_inner_wheel_link">
+    <material>Gazebo/DarkGrey</material>
+  </gazebo>
+  <gazebo reference="FR_outer_wheel_connector_link">
+    <material>Gazebo/Grey</material>
+  </gazebo>
+  <gazebo reference="FL_outer_wheel_connector_link">
+    <material>Gazebo/Grey</material>
+  </gazebo>
+  <gazebo reference="FR_inner_wheel_connector_link">
+    <material>Gazebo/Grey</material>
+  </gazebo>
+  <gazebo reference="FL_inner_wheel_connector_link">
+    <material>Gazebo/Grey</material>
+  </gazebo>
+  <gazebo reference="docker_link">
+    <material>Gazebo/Grey</material>
+  </gazebo>
+  <gazebo reference="R_docker_shaft_link">
+    <material>Gazebo/Red</material>
+  </gazebo>
+  <gazebo reference="L_docker_shaft_link">
+    <material>Gazebo/Red</material>
+  </gazebo>
 </robot>
